Commit message: working on the new model, with the control

File: wall_e_ws/src/wall_e_description/urdf/wall_e.gazebo.xacro (robot description, xacro)
@@ -1,78 +1,79 @@
-<?xml version="1.0" encoding="UTF-8"?>
 <robot name="wall_e" xmlns:xacro="http://www.ros.org/wiki/xacro">
-    <!--
-    <transmission name="front_wheel_right_transmission">
-        <plugin>transmission_interface/SimpleTransmission</plugin>
-        <joint name="front_right_wheel" role="joint_right">
-            <mechanical_reduction>1.0</mechanical_reduction>
+    <!-- Transmission for Front Right Wheel -->
+    <transmission name="FR_Transmission">
+        <type>transmission_interface/SimpleTransmission</type>
+        <joint name="FR_joint">
+            <hardwareInterface>hardware_interface/VelocityJointInterface</hardwareInterface>
         </joint>
-        <actuator name="front_right_wheel_motor" role="actuator_right"/>
+        <actuator name="FR_Motor">
+            <mechanicalReduction>1.0</mechanicalReduction>
+        </actuator>
     </transmission>
-    <transmission name="back_wheel_right_transmission">
-        <plugin>transmission_interface/SimpleTransmission</plugin>
-        <joint name="back_right_wheel" role="joint_right">
-            <mechanical_reduction>1.0</mechanical_reduction>
+    <!-- Transmission for Back Right Wheel -->
+    <transmission name="BR_Transmission">
+        <type>transmission_interface/SimpleTransmission</type>
+        <joint name="Br_joint">
+            <hardwareInterface>hardware_interface/VelocityJointInterface</hardwareInterface>
         </joint>
-        <actuator name="back_right_wheel_motor" role="actuator_right"/>
+        <actuator name="BR_Motor">
+            <mechanicalReduction>1.0</mechanicalReduction>
+        </actuator>
     </transmission>
-    <transmission name="front_wheel_left_transmission">
-        <plugin>transmission_interface/SimpleTransmission</plugin>
-        <joint name="front_left_wheel" role="joint_left">
-            <mechanical_reduction>1.0</mechanical_reduction>
+    <!-- Transmission for Front Left Wheel -->
+    <transmission name="FL_Transmission">
+        <type>transmission_interface/SimpleTransmission</type>
+        <joint name="FL_joint">
+            <hardwareInterface>hardware_interface/VelocityJointInterface</hardwareInterface>
         </joint>
-        <actuator name="front_left_wheel_motor" role="actuator_left"/>
+        <actuator name="FL_Motor">
+            <mechanicalReduction>1.0</mechanicalReduction>
+        </actuator>
     </transmission>
-    <transmission name="back_wheel_left_transmission">
-        <plugin>transmission_interface/SimpleTransmission</plugin>
-        <joint name="back_left_wheel" role="joint_left">
-            <mechanical_reduction>1.0</mechanical_reduction>
+    <!-- Transmission for Back Left Wheel -->
+    <transmission name="BL_Transmission">
+        <type>transmission_interface/SimpleTransmission</type>
+        <joint name="BL_joint">
+            <hardwareInterface>hardware_interface/VelocityJointInterface</hardwareInterface>
         </joint>
-        <actuator name="back_left_wheel_motor" role="actuator_left"/>
+        <actuator name="BL_Motor">
+            <mechanicalReduction>1.0</mechanicalReduction>
+        </actuator>
     </transmission>
-    -->
-    <gazebo reference="Front_Right_Wheel">
+  <!-- Gazebo configuration for left front wheel -->
+  <gazebo reference="FL_link">
         <mu1>100000000000000.0</mu1>
         <mu2>100000000000000.0</mu2>
         <kp>1000000000000.0</kp>
         <kd>10.0</kd>
-        <minDepth>0.001</minDepth>
-        <maxVel>0.1</maxVel>
-        <fdir1>1 0 0</fdir1>
-    </gazebo>
-    <gazebo reference="Front_Left_Wheel">
+  </gazebo>
+    <!-- Gazebo Friction Parameters for Front Right Wheel -->
+    <gazebo reference="FR_link">
         <mu1>100000000000000.0</mu1>
         <mu2>100000000000000.0</mu2>
         <kp>1000000000000.0</kp>
         <kd>10.0</kd>
-        <minDepth>0.001</minDepth>
-        <maxVel>0.1</maxVel>
-        <fdir1>1 0 0</fdir1>
-    </gazebo>
-    <gazebo reference="Back_Right_Wheel">
+      </gazebo>
+    <!-- Gazebo Friction Parameters for Back Left Wheel -->
+    <gazebo reference="BL_link">
         <mu1>100000000000000.0</mu1>
         <mu2>100000000000000.0</mu2>
         <kp>1000000000000.0</kp>
         <kd>10.0</kd>
-        <minDepth>0.001</minDepth>
-        <maxVel>0.1</maxVel>
-        <fdir1>1 0 0</fdir1>
-    </gazebo>
-    <gazebo reference="Back_Left_Wheel">
+      </gazebo>
+    <!-- Gazebo Friction Parameters for Back Right Wheel -->
+    <gazebo reference="BR_link">
         <mu1>100000000000000.0</mu1>
         <mu2>100000000000000.0</mu2>
         <kp>1000000000000.0</kp>
         <kd>10.0</kd>
-        <minDepth>0.001</minDepth>
-        <maxVel>0.1</maxVel>
-        <fdir1>1 0 0</fdir1>
-    </gazebo>
-    <!--
+      </gazebo>
+    <!-- Gazebo Plugin for ROS2 Control -->
     <gazebo>
         <plugin filename="libgazebo_ros2_control.so" name="gazebo_ros2_control">
             <robot_param>robot_description</robot_param>
             <robot_param_node>robot_state_publisher</robot_param_node>
-            <parameters>$(find bumperbot_controller)/config/bumperbot_controllers.yaml</parameters>
+            <!-- Correct the path to the YAML file -->
+            <parameters>$(find wall_e_controller)/config/wall_e_controllers.yaml</parameters>
         </plugin>
     </gazebo>
-    -->
 </robot>

File: wall_e_ws/src/wall_e_description/urdf/wall_e.urdf.xacro (robot description, xacro)
@@ -1,164 +1,263 @@
-<?xml version="1.0" encoding="utf-8"?>
-<!-- This URDF was automatically created by SolidWorks to URDF Exporter! Originally created by Stephen Brawner (brawner@gmail.com)
-     Commit Version: 1.6.0-4-g7f85cfe  Build Version: 1.6.7995.38578
-     For more information, please see http://wiki.ros.org/sw_urdf_exporter -->
 <robot xmlns:xacro="http://www.ros.org/wiki/xacro" name="wall_e">
   <xacro:include filename="$(find wall_e_description)/urdf/wall_e.gazebo.xacro"/>
+  <xacro:include filename="$(find wall_e_description)/urdf/wall_e_ros2_control.xacro"/>
   <link name="base_footprint">
-  </link>
-  <link name="base_link">
-    <inertial>
-      <origin xyz="0 0 0" rpy="0 0 0" />
-      <mass value="1.41415126127045" />
-      <inertia ixx="0.0102795735791383" ixy="1.27187727331604E-09" ixz="6.56701848981784E-08"
-        iyy="0.0129423397475402" iyz="2.60947122320625E-05" izz="0.00310768355824767" />
-    </inertial>
-    <visual>
-      <origin xyz="0 0 0" rpy="0 0 0" />
-      <geometry>
-        <mesh
-          filename="package://wall_e_description/meshes/Body.STL" />
-      </geometry>
-      <material name="">
-        <color rgba="0.792156862745098 0.819607843137255 0.933333333333333 1" />
-      </material>
-    </visual>
-    <collision>
-      <origin xyz="0 0 0" rpy="0 0 0" />
-      <geometry>
-        <mesh
-          filename="package://wall_e_description/meshes/Body.STL" />
-      </geometry>
-    </collision>
-  </link>
-  <link name="Front_Left_Wheel">
-    <inertial>
-      <origin xyz="5.55111512312578E-17 0.015 -5.55111512312578E-17" rpy="0 0 0" />
-      <mass value="0.104261024893665" />
-      <inertia ixx="3.75784516057514E-05" ixy="2.86174098456648E-22" ixz="0"
-        iyy="6.1107497194996E-05" iyz="1.37800244009481E-22" izz="3.75784516057514E-05" />
-    </inertial>
-    <visual>
-      <origin xyz="0 0 0" rpy="0 0 0" />
-      <geometry>
-        <mesh
-          filename="package://wall_e_description/meshes/Front_Left_Wheel.STL" />
-      </geometry>
-      <material name="">
-        <color rgba="0.792156862745098 0.819607843137255 0.933333333333333 1" />
-      </material>
-    </visual>
-    <collision>
-      <origin xyz="0 0 0" rpy="0 0 0" />
-      <geometry>
-        <sphere radius="0.033"/>
-      </geometry>
-    </collision>
-  </link>
-  <link name="Front_Right_Wheel">
-    <inertial>
-      <origin xyz="-5.55111512312578E-17 -0.015 1.38777878078145E-17" rpy="0 0 0" />
-      <mass value="0.104261024893665" />
-      <inertia ixx="3.75784516057513E-05" ixy="-1.74832828168085E-22" ixz="0"
-        iyy="6.1107497194996E-05" iyz="5.28856994197548E-22" izz="3.75784516057513E-05" />
-    </inertial>
-    <visual>
-      <origin xyz="0 0 0" rpy="0 0 0" />
-      <geometry>
-        <mesh filename="package://wall_e_description/meshes/Front_Right_Wheel.STL" />
-      </geometry>
-      <material name="">
-        <color rgba="0.792156862745098 0.819607843137255 0.933333333333333 1" />
-      </material>
-    </visual>
-    <collision>
-      <origin xyz="0 0 0" rpy="0 0 0" />
-      <geometry>
-        <sphere radius="0.033"/>
-      </geometry>
-    </collision>
-  </link>
-  <link name="Back_Left_Wheel">
-    <inertial>
-      <origin xyz="-2.08166817117217E-17 0.015 2.77555756156289E-17" rpy="0 0 0" />
-      <mass value="0.104261024893665" />
-      <inertia ixx="3.75784516057514E-05" ixy="2.79490905093828E-22" ixz="0"
-        iyy="6.1107497194996E-05" iyz="-3.36655961863459E-22" izz="3.75784516057514E-05" />
-    </inertial>
-    <visual>
-      <origin xyz="0 0 0" rpy="0 0 0" />
-      <geometry>
-        <mesh filename="package://wall_e_description/meshes/Back_Left_Wheel.STL" />
-      </geometry>
-      <material name="">
-        <color rgba="0.792156862745098 0.819607843137255 0.933333333333333 1" />
-      </material>
-    </visual>
-    <collision>
-      <origin xyz="0 0 0" rpy="0 0 0" />
-      <geometry>
-        <sphere radius="0.033"/>
-      </geometry>
-    </collision>
-  </link>
-  <link name="Back_Right_Wheel">
-    <inertial>
-      <origin xyz="0 -0.015 6.93889390390723E-18" rpy="0 0 0" />
-      <mass value="0.104261024893665" />
-      <inertia ixx="3.75784516057514E-05" ixy="5.44261580910539E-24" ixz="0"
-        iyy="6.1107497194996E-05" iyz="-2.9089336076258E-23" izz="3.75784516057514E-05" />
-    </inertial>
-    <visual>
-      <origin xyz="0 0 0" rpy="0 0 0" />
-      <geometry>
-        <mesh filename="package://wall_e_description/meshes/Back_Right_Wheel.STL" />
-      </geometry>
-      <material name="">
-        <color rgba="0.792156862745098 0.819607843137255 0.933333333333333 1" />
-      </material>
-    </visual>
-    <collision>
-      <origin xyz="0 0 0" rpy="0 0 0" />
-      <geometry>
-        <sphere radius="0.033"/>
-      </geometry>
-    </collision>
   </link>
   <joint name="base_joint" type="fixed">
     <parent link="base_footprint"/>
     <child link="base_link"/>
-    <origin rpy="0 0 3.14" xyz="0 0 0.033"/>
-  </joint>
-  <joint name="front_left_wheel" type="continuous">
-    <origin xyz="0.11285 -0.16498 0.048102" rpy="3.1416 0.87981 1.5708" />
-    <parent link="base_link" />
-    <child link="Front_Left_Wheel" />
-    <axis xyz="0 1 0" />
-    <limit effort="10" velocity="10" />
-    <dynamics damping="0.1" friction="0.1" />
-  </joint>
-  <joint name="front_right_wheel" type="continuous">
-    <origin xyz="-0.08301 -0.16498 0.048102" rpy="3.1416 0.49133 1.5708" />
-    <parent link="base_link" />
-    <child link="Front_Right_Wheel" />
-    <axis xyz="0 1 0" />
-    <limit effort="10" velocity="10" />
-    <dynamics damping="0.1" friction="0.1" />
-  </joint>
-  <joint name="back_left_wheel" type="continuous">
-    <origin xyz="0.11285 0.027952 0.048102" rpy="3.1416 0.81738 1.5708" />
-    <parent link="base_link" />
-    <child link="Back_Left_Wheel" />
-    <axis xyz="0 1 0" />
-    <limit effort="10" velocity="10" />
-    <dynamics damping="0.1" friction="0.1" />
-  </joint>
-  <joint name="back_right_wheel" type="continuous">
-    <origin xyz="-0.08301 0.027952 0.048102" rpy="3.1416 0.92219 1.5708" />
-    <parent link="base_link" />
-    <child link="Back_Right_Wheel" />
-    <axis xyz="0 1 0" />
-    <limit effort="10" velocity="10" />
-    <dynamics damping="0.1" friction="0.1" />
+    <origin rpy="0 0 0" xyz="0 0 0.02"/>
+  </joint>
+  <link
+    name="base_link">
+    <inertial>
+      <origin
+        xyz="0.0155792528368141 -3.13584449863485E-05 -0.043885278180218"
+        rpy="0 0 0" />
+      <mass
+        value="7.30051365588478" />
+      <inertia
+        ixx="0.0307878292952919"
+        ixy="-7.35451053591693E-06"
+        ixz="1.00519054145349E-05"
+        iyy="0.0629723510018648"
+        iyz="-8.74590698168669E-07"
+        izz="0.0877757846541169" />
+    </inertial>
+    <visual>
+      <origin
+        xyz="0 0 0"
+        rpy="0 0 0" />
+      <geometry>
+        <mesh
+          filename="package://wall_e_description/meshes/base_link.STL" />
+      </geometry>
+      <material
+        name="">
+        <color
+          rgba="0.752941176470588 0.752941176470588 0.752941176470588 1" />
+      </material>
+    </visual>
+    <collision>
+      <origin
+        xyz="0 0 0"
+        rpy="0 0 0" />
+      <geometry>
+        <mesh
+          filename="package://wall_e_description/meshes/base_link.STL" />
+      </geometry>
+    </collision>
+  </link>
+  <link
+    name="BR_link">
+    <inertial>
+      <origin
+        xyz="2.9442E-08 0.05681 -1.1142E-07"
+        rpy="0 0 0" />
+      <mass
+        value="0.70354" />
+      <inertia
+        ixx="0.00045383"
+        ixy="2.2319E-09"
+        ixz="-2.0047E-08"
+        iyy="0.00059175"
+        iyz="-2.9703E-09"
+        izz="0.00045385" />
+    </inertial>
+    <visual>
+      <origin
+        xyz="0 0 0"
+        rpy="0 0 0" />
+      <geometry>
+        <mesh
+          filename="package://wall_e_description/meshes/BR_link.STL" />
+      </geometry>
+      <material
+        name="">
+        <color
+          rgba="0.75294 0.75294 0.75294 1" />
+      </material>
+    </visual>
+    <collision>
+      <origin
+        xyz="0 0 0"
+        rpy="0 0 0" />
+      <geometry>
+        <mesh
+          filename="package://wall_e_description/meshes/BR_link.STL" />
+      </geometry>
+    </collision>
+  </link>
+  <joint
+    name="BR_joint"
+    type="continuous">
+    <origin
+      xyz="-0.26698 -0.2513 -0.1585"
+      rpy="0 0 0" />
+    <parent
+      link="base_link" />
+    <child
+      link="BR_link" />
+    <axis
+      xyz="0 1 0" />
+  </joint>
+  <link
+    name="FR_link">
+    <inertial>
+      <origin
+        xyz="-1.3001E-07 0.05681 -1.2687E-07"
+        rpy="0 0 0" />
+      <mass
+        value="0.70354" />
+      <inertia
+        ixx="0.00045383"
+        ixy="-6.1874E-10"
+        ixz="2.0686E-08"
+        iyy="0.00059175"
+        iyz="-2.702E-09"
+        izz="0.00045385" />
+    </inertial>
+    <visual>
+      <origin
+        xyz="0 0 0"
+        rpy="0 0 0" />
+      <geometry>
+        <mesh
+          filename="package://wall_e_description/meshes/FR_link.STL"  />
+      </geometry>
+      <material
+        name="">
+        <color
+          rgba="0.75294 0.75294 0.75294 1" />
+      </material>
+    </visual>
+    <collision>
+      <origin
+        xyz="0 0 0"
+        rpy="0 0 0" />
+      <geometry>
+        <mesh
+          filename="package://wall_e_description/meshes/FR_link.STL"  />
+      </geometry>
+    </collision>
+  </link>
+  <joint
+    name="FR_joint"
+    type="continuous">
+    <origin
+      xyz="0.28978 -0.2513 -0.1585"
+      rpy="0 0 0" />
+    <parent
+      link="base_link" />
+    <child
+      link="FR_link" />
+    <axis
+      xyz="0 1 0" />
+  </joint>
+  <link
+    name="FL_link">
+    <inertial>
+      <origin
+        xyz="1.3043E-07 -0.05681 1.2701E-07"
+        rpy="0 0 0" />
+      <mass
+        value="0.70354" />
+      <inertia
+        ixx="0.00045383"
+        ixy="-6.7038E-10"
+        ixz="2E-08"
+        iyy="0.00059175"
+        iyz="-2.7151E-09"
+        izz="0.00045385" />
+    </inertial>
+    <visual>
+      <origin
+        xyz="0 0 0"
+        rpy="0 0 0" />
+      <geometry>
+        <mesh
+          filename="package://wall_e_description/meshes/FL_link.STL" />
+      </geometry>
+      <material
+        name="">
+        <color
+          rgba="0.75294 0.75294 0.75294 1" />
+      </material>
+    </visual>
+    <collision>
+      <origin
+        xyz="0 0 0"
+        rpy="0 0 0" />
+      <geometry>
+        <mesh
+          filename="package://wall_e_description/meshes/FL_link.STL" />
+      </geometry>
+    </collision>
+  </link>
+  <joint
+    name="FL_joint"
+    type="continuous">
+    <origin
+      xyz="0.28978 0.2515 -0.1585"
+      rpy="0 0 0" />
+    <parent
+      link="base_link" />
+    <child
+      link="FL_link" />
+    <axis
+      xyz="0 1 0" />
+  </joint>
+  <link
+    name="BL_link">
+    <inertial>
+      <origin
+        xyz="1.2093E-07 -0.05681 -1.6462E-07"
+        rpy="0 0 0" />
+      <mass
+        value="0.70354" />
+      <inertia
+        ixx="0.00045383"
+        ixy="-8.0131E-10"
+        ixz="-2.0772E-08"
+        iyy="0.00059175"
+        iyz="2.1066E-09"
+        izz="0.00045385" />
+    </inertial>
+    <visual>
+      <origin
+        xyz="0 0 0"
+        rpy="0 0 0" />
+      <geometry>
+        <mesh
+          filename="package://wall_e_description/meshes/BL_link.STL" />
+      </geometry>
+      <material
+        name="">
+        <color
+          rgba="0.75294 0.75294 0.75294 1" />
+      </material>
+    </visual>
+    <collision>
+      <origin
+        xyz="0 0 0"
+        rpy="0 0 0" />
+      <geometry>
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
Commit message: I love you peter

File: wall_e_ws/src/wall_e_description/urdf/wall_e.gazebo.xacro (robot description, xacro)
@@ -77,3 +77,80 @@
         </plugin>
     </gazebo>
-</robot>
+<gazebo reference="imu_link">
+      <sensor name="imu" type="imu">
+          <always_on>true</always_on>
+          <update_rate>100</update_rate>
+          <imu>
+            <angular_velocity>
+              <x>
+                <noise type="gaussian">
+                  <mean>0.0</mean>
+                  <stddev>2e-4</stddev>
+                </noise>
+              </x>
+              <y>
+                <noise type="gaussian">
+                  <mean>0.0</mean>
+                  <stddev>2e-4</stddev>
+                </noise>
+              </y>
+              <z>
+                <noise type="gaussian">
+                  <mean>0.0</mean>
+                  <stddev>2e-4</stddev>
+                </noise>
+              </z>
+            </angular_velocity>
+            <linear_acceleration>
+              <x>
+                <noise type="gaussian">
+                  <mean>0.0</mean>
+                  <stddev>1.7e-2</stddev>
+                </noise>
+              </x>
+              <y>
+                <noise type="gaussian">
+                  <mean>0.0</mean>
+                  <stddev>1.7e-2</stddev>
+                </noise>
+              </y>
+              <z>
+                <noise type="gaussian">
+                  <mean>0.0</mean>
+                  <stddev>1.7e-2</stddev>
+                </noise>
+              </z>
+            </linear_acceleration>
+          </imu>
+          <plugin name="imu" filename="libgazebo_ros_imu_sensor.so"/>
+      </sensor>
+</gazebo>
+ <gazebo reference="gps_link">
+      <sensor name="tb3_gps" type="gps">
+        <always_on>true</always_on>
+        <update_rate>1</update_rate>
+        <pose>0 0 0 0 0 0</pose>
+        <gps>
+          <position_sensing>
+            <horizontal>
+              <noise type="gaussian">
+                <mean>0.0</mean>
+                <stddev>0.01</stddev>
+              </noise>
+            </horizontal>
+            <vertical>
+              <noise type="gaussian">
+                <mean>0.0</mean>
+                <stddev>0.01</stddev>
+              </noise>
+            </vertical>
+          </position_sensing>
+        </gps>
+        <plugin name="my_gps_plugin" filename="libgazebo_ros_gps_sensor.so">
+          <ros>
+            <remapping>~/out:=/gps/fix</remapping>
+          </ros>
+        </plugin>
+      </sensor>
+    </gazebo>
+    </robot>

File: wall_e_ws/src/wall_e_description/urdf/wall_e.urdf.xacro (robot description, xacro)
@@ -261,3 +261,37 @@
       xyz="0 1 0" />
   </joint>
-</robot>
+ <joint name="imu_joint" type="fixed">
+        <parent link="base_link"/>
+        <child link="imu_link"/>
+        <origin xyz="0 0 0.7" rpy="0 0 0"/>
+        <axis xyz="0 0 0"/>
+    </joint>
+ <link name="imu_link">
+        <inertial>
+            <origin xyz="-0.00552433659106688 0.000168210391520346 0.000514000497342681" rpy="0 0 0" />
+            <mass value="0.000528415362211671" />
+            <inertia ixx="1.46176048428261E-08" ixy="1.40015117949421E-10" ixz="-1.99633872937403E-12"
+                     iyy="8.59662482954888E-09" iyz="7.52375112767959E-12"
+                     izz="2.30279421279312E-08" />
+        </inertial>
+        <visual>
+            <origin xyz="0 0 0" rpy="0 0 0"/>
+            <geometry>
+                <mesh filename="package://wall_e_description/meshes/imu_link.STL"/>
+            </geometry>
+        </visual>
+        <collision>
+            <origin xyz="0 0 0" rpy="0 0 0"/>
+            <geometry>
+                <mesh filename="package://wall_e_description/meshes/imu_link.STL"/>
+            </geometry>
+        </collision>
+    </link>
+    <link name="gps_link"/>
+    <!-- Add the gps link so we get a static transform for the GPS -->
+    <joint name="gps_joint" type="fixed">
+      <parent link="base_link"/>
+      <child link="gps_link"/>
+      <origin xyz="0 0 0" rpy="0 0 0"/>
+    </joint>
+    </robot>
