Commit message: trying working model

File: wall_e_ws/src/wall_e_description/urdf/wall_e.gazebo.xacro (robot description, xacro)
@@ -13,5 +13,5 @@
     <transmission name="BR_Transmission">
         <type>transmission_interface/SimpleTransmission</type>
-        <joint name="Br_joint">
+        <joint name="BR_joint">
             <hardwareInterface>hardware_interface/VelocityJointInterface</hardwareInterface>
         </joint>

File: wall_e_ws/src/wall_e_description/urdf/wall_e.urdf.xacro (robot description, xacro)
@@ -13,15 +13,15 @@
     <inertial>
       <origin
-        xyz="0.0155792528368141 -3.13584449863485E-05 -0.043885278180218"
-        rpy="0 0 0" />
-      <mass
-        value="7.30051365588478" />
-      <inertia
-        ixx="0.0307878292952919"
-        ixy="-7.35451053591693E-06"
-        ixz="1.00519054145349E-05"
-        iyy="0.0629723510018648"
-        iyz="-8.74590698168669E-07"
-        izz="0.0877757846541169" />
+        xyz="0.00809763256593836 -0.000562322358044154 -0.0289427041542462"
+        rpy="0 0 0" />
+      <mass
+        value="0.98435044127488" />
+      <inertia
+        ixx="0.00719634458823369"
+        ixy="-2.65438242709729E-09"
+        ixz="3.80350663889404E-08"
+        iyy="0.00694500656023865"
+        iyz="-1.52985888763549E-09"
+        izz="0.0123629441660506" />
     </inertial>
     <visual>
@@ -53,15 +53,15 @@
     <inertial>
       <origin
-        xyz="2.9442E-08 0.05681 -1.1142E-07"
-        rpy="0 0 0" />
-      <mass
-        value="0.70354" />
-      <inertia
-        ixx="0.00045383"
-        ixy="2.2319E-09"
-        ixz="-2.0047E-08"
-        iyy="0.00059175"
-        iyz="-2.9703E-09"
-        izz="0.00045385" />
+        xyz="0 0.02152 0"
+        rpy="0 0 0" />
+      <mass
+        value="0.42795" />
+      <inertia
+        ixx="0.00040313"
+        ixy="4.2213E-22"
+        ixz="-2.2648E-36"
+        iyy="0.00067844"
+        iyz="9.9268E-21"
+        izz="0.00040313" />
     </inertial>
     <visual>
@@ -93,5 +93,5 @@
     type="continuous">
     <origin
-      xyz="-0.26698 -0.2513 -0.1585"
+      xyz="-0.082838 -0.1596 -0.1041"
       rpy="0 0 0" />
     <parent
@@ -106,37 +106,37 @@
     <inertial>
       <origin
-        xyz="-1.3001E-07 0.05681 -1.2687E-07"
-        rpy="0 0 0" />
-      <mass
-        value="0.70354" />
-      <inertia
-        ixx="0.00045383"
-        ixy="-6.1874E-10"
-        ixz="2.0686E-08"
-        iyy="0.00059175"
-        iyz="-2.702E-09"
-        izz="0.00045385" />
-    </inertial>
-    <visual>
-      <origin
-        xyz="0 0 0"
-        rpy="0 0 0" />
-      <geometry>
-        <mesh
-          filename="package://wall_e_description/meshes/FR_link.STL"  />
-      </geometry>
-      <material
-        name="">
-        <color
-          rgba="0.75294 0.75294 0.75294 1" />
-      </material>
-    </visual>
-    <collision>
-      <origin
-        xyz="0 0 0"
-        rpy="0 0 0" />
-      <geometry>
-        <mesh
-          filename="package://wall_e_description/meshes/FR_link.STL"  />
+        xyz="2.7756E-17 0.02152 0"
+        rpy="0 0 0" />
+      <mass
+        value="0.42795" />
+      <inertia
+        ixx="0.00040313"
+        ixy="4.5137E-22"
+        ixz="-1.0801E-37"
+        iyy="0.00067844"
+        iyz="9.9268E-21"
+        izz="0.00040313" />
+    </inertial>
+    <visual>
+      <origin
+        xyz="0 0 0"
+        rpy="0 0 0" />
+      <geometry>
+        <mesh
+          filename="package://wall_e_description/meshes/FR_link.STL" />
+      </geometry>
+      <material
+        name="">
+        <color
+          rgba="0.75294 0.75294 0.75294 1" />
+      </material>
+    </visual>
+    <collision>
+      <origin
+        xyz="0 0 0"
+        rpy="0 0 0" />
+      <geometry>
+        <mesh
+          filename="package://wall_e_description/meshes/FR_link.STL" />
       </geometry>
     </collision>
@@ -146,5 +146,5 @@
     type="continuous">
     <origin
-      xyz="0.28978 -0.2513 -0.1585"
+      xyz="0.082849 -0.1596 -0.1041"
       rpy="0 0 0" />
     <parent
@@ -159,15 +159,15 @@
     <inertial>
       <origin
-        xyz="1.3043E-07 -0.05681 1.2701E-07"
-        rpy="0 0 0" />
-      <mass
-        value="0.70354" />
-      <inertia
-        ixx="0.00045383"
-        ixy="-6.7038E-10"
-        ixz="2E-08"
-        iyy="0.00059175"
-        iyz="-2.7151E-09"
-        izz="0.00045385" />
+        xyz="2.7756E-17 -0.02152 0"
+        rpy="0 0 0" />
+      <mass
+        value="0.42795" />
+      <inertia
+        ixx="0.00040313"
+        ixy="2.1117E-21"
+        ixz="-2.9719E-20"
+        iyy="0.00067844"
+        iyz="-7.8622E-21"
+        izz="0.00040313" />
     </inertial>
     <visual>
@@ -199,5 +199,5 @@
     type="continuous">
     <origin
-      xyz="0.28978 0.2515 -0.1585"
+      xyz="0.082849 0.1596 -0.1041"
       rpy="0 0 0" />
     <parent
@@ -212,15 +212,15 @@
     <inertial>
       <origin
-        xyz="1.2093E-07 -0.05681 -1.6462E-07"
-        rpy="0 0 0" />
-      <mass
-        value="0.70354" />
-      <inertia
-        ixx="0.00045383"
-        ixy="-8.0131E-10"
-        ixz="-2.0772E-08"
-        iyy="0.00059175"
-        iyz="2.1066E-09"
-        izz="0.00045385" />
+        xyz="0 -0.02152 0"
+        rpy="0 0 0" />
+      <mass
+        value="0.42795" />
+      <inertia
+        ixx="0.00040313"
+        ixy="3.055E-21"
+        ixz="-2.4304E-20"
+        iyy="0.00067844"
+        iyz="-8.2856E-21"
+        izz="0.00040313" />
     </inertial>
     <visual>
@@ -252,5 +252,5 @@
     type="continuous">
     <origin
-      xyz="-0.26698 0.2515 -0.1585"
+      xyz="-0.082838 0.1596 -0.1041"
       rpy="0 0 0" />
     <parent

Commit message: playing with the urdf and nav2 as well as the controller

File: wall_e_ws/src/wall_e_description/urdf/wall_e.gazebo.xacro (robot description, xacro)
@@ -40,41 +40,4 @@
         </actuator>
     </transmission>
-  <!-- Gazebo configuration for left front wheel -->
-  <gazebo reference="FL_link">
-        <mu1>100000000000000.0</mu1>
-        <mu2>100000000000000.0</mu2>
-        <kp>1000000000000.0</kp>
-        <kd>10.0</kd>
-  </gazebo>
-    <!-- Gazebo Friction Parameters for Front Right Wheel -->
-    <gazebo reference="FR_link">
-        <mu1>100000000000000.0</mu1>
-        <mu2>100000000000000.0</mu2>
-        <kp>1000000000000.0</kp>
-        <kd>10.0</kd>
-      </gazebo>
-    <!-- Gazebo Friction Parameters for Back Left Wheel -->
-    <gazebo reference="BL_link">
-        <mu1>100000000000000.0</mu1>
-        <mu2>100000000000000.0</mu2>
-        <kp>1000000000000.0</kp>
-        <kd>10.0</kd>
-      </gazebo>
-    <!-- Gazebo Friction Parameters for Back Right Wheel -->
-    <gazebo reference="BR_link">
-        <mu1>100000000000000.0</mu1>
-        <mu2>100000000000000.0</mu2>
-        <kp>1000000000000.0</kp>
-        <kd>10.0</kd>
-      </gazebo>
-    <!-- Gazebo Plugin for ROS2 Control -->
-    <gazebo>
-        <plugin filename="libgazebo_ros2_control.so" name="gazebo_ros2_control">
-            <robot_param>robot_description</robot_param>
-            <robot_param_node>robot_state_publisher</robot_param_node>
-            <!-- Correct the path to the YAML file -->
-            <parameters>$(find wall_e_controller)/config/wall_e_controllers.yaml</parameters>
-        </plugin>
-    </gazebo>
 <gazebo reference="imu_link">
       <sensor name="imu" type="imu">

File: wall_e_ws/src/wall_e_description/urdf/wall_e.urdf.xacro (robot description, xacro)
@@ -13,15 +13,15 @@
     <inertial>
       <origin
-        xyz="0.00809763256593836 -0.000562322358044154 -0.0289427041542462"
-        rpy="0 0 0" />
-      <mass
-        value="0.98435044127488" />
-      <inertia
-        ixx="0.00719634458823369"
-        ixy="-2.65438242709729E-09"
-        ixz="3.80350663889404E-08"
-        iyy="0.00694500656023865"
-        iyz="-1.52985888763549E-09"
-        izz="0.0123629441660506" />
+        xyz="2.12503625807159E-17 0 -0.0212688653283583"
+        rpy="0 0 0" />
+      <mass
+        value="19.7944372375747" />
+      <inertia
+        ixx="0.236926173828267"
+        ixy="2.08285401729832E-18"
+        ixz="3.25260651745651E-19"
+        iyy="0.335947375820388"
+        iyz="7.19978005166155E-21"
+        izz="0.566141968007365" />
     </inertial>
     <visual>
@@ -50,53 +50,53 @@
   </link>
   <link
-    name="BR_link">
-    <inertial>
-      <origin
-        xyz="0 0.02152 0"
-        rpy="0 0 0" />
-      <mass
-        value="0.42795" />
-      <inertia
-        ixx="0.00040313"
-        ixy="4.2213E-22"
-        ixz="-2.2648E-36"
-        iyy="0.00067844"
-        iyz="9.9268E-21"
-        izz="0.00040313" />
-    </inertial>
-    <visual>
-      <origin
-        xyz="0 0 0"
-        rpy="0 0 0" />
-      <geometry>
-        <mesh
-          filename="package://wall_e_description/meshes/BR_link.STL" />
-      </geometry>
-      <material
-        name="">
-        <color
-          rgba="0.75294 0.75294 0.75294 1" />
-      </material>
-    </visual>
-    <collision>
-      <origin
-        xyz="0 0 0"
-        rpy="0 0 0" />
-      <geometry>
-        <mesh
-          filename="package://wall_e_description/meshes/BR_link.STL" />
+    name="FL_link">
+    <inertial>
+      <origin
+        xyz="-2.7756E-16 -0.049964 -1.9915E-15"
+        rpy="0 0 0" />
+      <mass
+        value="1.7656" />
+      <inertia
+        ixx="0.0039551"
+        ixy="1.3837E-18"
+        ixz="-2.0269E-19"
+        iyy="0.0049701"
+        iyz="1.6232E-18"
+        izz="0.0039551" />
+    </inertial>
+    <visual>
+      <origin
+        xyz="0 0 0"
+        rpy="0 0 0" />
+      <geometry>
+        <mesh
+          filename="package://wall_e_description/meshes/FL_link.STL" />
+      </geometry>
+      <material
+        name="">
+        <color
+          rgba="0.29804 0.29804 0.29804 1" />
+      </material>
+    </visual>
+    <collision>
+      <origin
+        xyz="0 0 0"
+        rpy="0 0 0" />
+      <geometry>
+        <mesh
+          filename="package://wall_e_description/meshes/FL_link.STL" />
       </geometry>
     </collision>
   </link>
   <joint
-    name="BR_joint"
+    name="FL_joint"
     type="continuous">
     <origin
-      xyz="-0.082838 -0.1596 -0.1041"
-      rpy="0 0 0" />
-    <parent
-      link="base_link" />
-    <child
-      link="BR_link" />
+      xyz="0.31152 0.302 -0.099351"
+      rpy="0 0 0" />
+    <parent
+      link="base_link" />
+    <child
+      link="FL_link" />
     <axis
       xyz="0 1 0" />
@@ -106,15 +106,15 @@
     <inertial>
       <origin
-        xyz="2.7756E-17 0.02152 0"
-        rpy="0 0 0" />
-      <mass
-        value="0.42795" />
-      <inertia
-        ixx="0.00040313"
-        ixy="4.5137E-22"
-        ixz="-1.0801E-37"
-        iyy="0.00067844"
-        iyz="9.9268E-21"
-        izz="0.00040313" />
+        xyz="0 0.049964 6.9389E-18"
+        rpy="0 0 0" />
+      <mass
+        value="1.7656" />
+      <inertia
+        ixx="0.0039551"
+        ixy="-7.6372E-19"
+        ixz="1.5112E-19"
+        iyy="0.0049701"
+        iyz="-1.9258E-19"
+        izz="0.0039551" />
     </inertial>
     <visual>
@@ -129,5 +129,5 @@
         name="">
         <color
-          rgba="0.75294 0.75294 0.75294 1" />
+          rgba="0.29804 0.29804 0.29804 1" />
       </material>
     </visual>
@@ -146,5 +146,5 @@
     type="continuous">
     <origin
-      xyz="0.082849 -0.1596 -0.1041"
+      xyz="0.31152 -0.302 -0.099351"
       rpy="0 0 0" />
     <parent
@@ -156,71 +156,18 @@
   </joint>
   <link
-    name="FL_link">
-    <inertial>
-      <origin
-        xyz="2.7756E-17 -0.02152 0"
-        rpy="0 0 0" />
-      <mass
-        value="0.42795" />
-      <inertia
-        ixx="0.00040313"
-        ixy="2.1117E-21"
-        ixz="-2.9719E-20"
-        iyy="0.00067844"
-        iyz="-7.8622E-21"
-        izz="0.00040313" />
-    </inertial>
-    <visual>
-      <origin
-        xyz="0 0 0"
-        rpy="0 0 0" />
-      <geometry>
-        <mesh
-          filename="package://wall_e_description/meshes/FL_link.STL" />
-      </geometry>
-      <material
-        name="">
-        <color
-          rgba="0.75294 0.75294 0.75294 1" />
-      </material>
-    </visual>
-    <collision>
-      <origin
-        xyz="0 0 0"
-        rpy="0 0 0" />
-      <geometry>
-        <mesh
-          filename="package://wall_e_description/meshes/FL_link.STL" />
-      </geometry>
-    </collision>
-  </link>
-  <joint
-    name="FL_joint"
-    type="continuous">
-    <origin
-      xyz="0.082849 0.1596 -0.1041"
-      rpy="0 0 0" />
-    <parent
-      link="base_link" />
-    <child
-      link="FL_link" />
-    <axis
-      xyz="0 1 0" />
-  </joint>
-  <link
     name="BL_link">
     <inertial>
       <origin
-        xyz="0 -0.02152 0"
-        rpy="0 0 0" />
-      <mass
-        value="0.42795" />
-      <inertia
-        ixx="0.00040313"
-        ixy="3.055E-21"
-        ixz="-2.4304E-20"
-        iyy="0.00067844"
-        iyz="-8.2856E-21"
-        izz="0.00040313" />
+        xyz="5.5511E-17 -0.049964 6.9389E-18"
+        rpy="0 0 0" />
+      <mass
+        value="1.7656" />
+      <inertia
+        ixx="0.0039551"
+        ixy="2.3359E-19"
+        ixz="-5.627E-20"
+        iyy="0.0049701"
+        iyz="-5.1707E-20"
+        izz="0.0039551" />
     </inertial>
     <visual>
@@ -235,5 +182,5 @@
         name="">
         <color
-          rgba="0.75294 0.75294 0.75294 1" />
+          rgba="0.29804 0.29804 0.29804 1" />
       </material>
     </visual>
@@ -252,5 +199,5 @@
     type="continuous">
     <origin
-      xyz="-0.082838 0.1596 -0.1041"
+      xyz="-0.31152 0.302 -0.099351"
       rpy="0 0 0" />
     <parent
@@ -261,31 +208,133 @@
       xyz="0 1 0" />
   </joint>
- <joint name="imu_joint" type="fixed">
-        <parent link="base_link"/>
-        <child link="imu_link"/>
-        <origin xyz="0 0 0.7" rpy="0 0 0"/>
-        <axis xyz="0 0 0"/>
-    </joint>
- <link name="imu_link">
-        <inertial>
-            <origin xyz="-0.00552433659106688 0.000168210391520346 0.000514000497342681" rpy="0 0 0" />
-            <mass value="0.000528415362211671" />
-            <inertia ixx="1.46176048428261E-08" ixy="1.40015117949421E-10" ixz="-1.99633872937403E-12"
-                     iyy="8.59662482954888E-09" iyz="7.52375112767959E-12"
-                     izz="2.30279421279312E-08" />
-        </inertial>
-        <visual>
-            <origin xyz="0 0 0" rpy="0 0 0"/>
-            <geometry>
-                <mesh filename="package://wall_e_description/meshes/imu_link.STL"/>
-            </geometry>
-        </visual>
-        <collision>
-            <origin xyz="0 0 0" rpy="0 0 0"/>
-            <geometry>
-                <mesh filename="package://wall_e_description/meshes/imu_link.STL"/>
-            </geometry>
-        </collision>
-    </link>
+  <link
+    name="BR_link">
+    <inertial>
+      <origin
+        xyz="5.5511E-17 0.049964 -6.9389E-18"
+        rpy="0 0 0" />
+      <mass
+        value="1.7656" />
+      <inertia
+        ixx="0.0039551"
+        ixy="6.4164E-19"
+        ixz="5.5883E-20"
+        iyy="0.0049701"
+        iyz="-1.0198E-19"
+        izz="0.0039551" />
+    </inertial>
+    <visual>
+      <origin
+        xyz="0 0 0"
+        rpy="0 0 0" />
+      <geometry>
+        <mesh
+          filename="package://wall_e_description/meshes/BR_link.STL" />
+      </geometry>
+      <material
+        name="">
+        <color
+          rgba="0.29804 0.29804 0.29804 1" />
+      </material>
+    </visual>
+    <collision>
+      <origin
+        xyz="0 0 0"
+        rpy="0 0 0" />
+      <geometry>
+        <mesh
+          filename="package://wall_e_description/meshes/BR_link.STL" />
+      </geometry>
+    </collision>
+  </link>
+    <joint
+    name="BR_joint"
+    type="continuous">
+    <origin
+      xyz="-0.31152 -0.302 -0.099351"
+      rpy="0 0 0" />
+    <parent
+      link="base_link" />
+    <child
+      link="BR_link" />
+    <axis
+      xyz="0 1 0" />
+  </joint>
+    <gazebo>
+    <plugin filename="libgazebo_ros_diff_drive.so" name="skid_steer_drive">
+      <!-- Update rate -->
+      <update_rate>500</update_rate>
+      <!-- Number of wheel pairs -->
+      <num_wheel_pairs>2</num_wheel_pairs>
+      <!-- wheels0 -->
+      <left_joint>FL_joint</left_joint>
+      <right_joint>FR_joint</right_joint>
+      <!-- wheels1-->
+      <left_joint>BL_joint</left_joint>
+      <right_joint>BR_joint</right_joint>
+      <!-- kinematics -->
+      <wheel_separation>0.33</wheel_separation>
+      <wheel_separation>0.33</wheel_separation>
+      <wheel_diameter>0.152</wheel_diameter>
+      <wheel_diameter>0.152</wheel_diameter>
+      <!-- limits -->
+      <max_wheel_torque>200</max_wheel_torque>
+      <max_wheel_acceleration>10.0</max_wheel_acceleration>
+      <!-- output -->
+      <odometry_frame>odom</odometry_frame>
+      <robot_base_frame>base_footprint</robot_base_frame>
+      <publish_odom>true</publish_odom>
+      <publish_odom_tf>true</publish_odom_tf>
+      <publish_wheel_tf>true</publish_wheel_tf>
+    </plugin>
+  </gazebo>
+  <link
+    name="IMU_link">
+    <inertial>
+      <origin
+        xyz="-4.3368E-19 -1.7347E-18 -0.005"
+        rpy="0 0 0" />
+      <mass
+        value="0.089" />
+      <inertia
+        ixx="1.9283E-05"
+        ixy="0"
+        ixz="0"
+        iyy="3.7083E-06"
+        iyz="-4.7189E-39"
+        izz="2.1508E-05" />
+    </inertial>
+    <visual>
+      <origin
+        xyz="0 0 0"
+        rpy="0 0 0" />
+      <geometry>
+        <mesh
+          filename="package://wall_e_description/meshes/IMU_link.STL" />
+      </geometry>
+    </visual>
+    <collision>
+      <origin
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